File: Precision Analog Isolation Amplifier/Precision Analog Isolation Amplifier.kicad_pcb (KiCad board)
At the start: 2 copper layers, 63.5 x 44 mm, 63 parts, among them IC1 ADA4899-1YRDZ, J1 Conn_01x03, J2 Conn_01x03, J3 Conn_Coaxial, J4 Conn_Coaxial, Q1 ---, U1 HCNR201, U2 ADA4522, U4 ADA4522

Commit message: Update PCB & Schematic
Parts:
- removed REF** (x4): MountingHole_2.2mm_M2_DIN965_Pad, MountingHole:MountingHole_2.2mm_M2_DIN965_Pad
- moved IC1 1.66 mm to (160.0, 115.0)
Connections:
- J3 pad 3: (no net) -> GND1
- J3 pad 4: (no net) -> GND1
- J3 pad 5: (no net) -> GND1
- J4 pad 3: (no net) -> GND2
- J4 pad 4: (no net) -> GND2
- J4 pad 5: (no net) -> GND2
- U2 pad 5: unconnected-(U2B-+-Pad5) -> GND2
- U2 pad 6: unconnected-(U2B---Pad6) -> Net-(U2B--)
- U2 pad 7: unconnected-(U2-Pad7) -> Net-(U2B--)
- U4 pad 5: unconnected-(U4B-+-Pad5) -> GND1
- U4 pad 6: unconnected-(U4B---Pad6) -> Net-(U4B--)
- U4 pad 7: unconnected-(U4-Pad7) -> Net-(U4B--)
Routing:
- net GND2: track 117.3 -> 138.8 mm
- net GND1: track 111.4 -> 125.6 mm, vias 8 -> 6
- net VEE2 -15V: track 30.7 -> 42.6 mm, vias 2 -> 3
- net Net-(U1B-K): track 49.4 -> 59.1 mm, vias 4 -> 2
- net Net-(IC1-+IN): track 6.83 -> 3.40 mm, vias 2 -> 0
- net Vout: track 26.8 -> 29.8 mm
- net Net-(U4B--): track 0.00 -> 1.27 mm
- net Net-(U2B--): track 0.00 -> 1.27 mm

Commit message: Commit
Parts:
- added REF**: MountingHole_3.2mm_M3, MountingHole:MountingHole_3.2mm_M3, F.Cu at (114.3, 79.9)
- added REF**: MountingHole_3.2mm_M3, MountingHole:MountingHole_3.2mm_M3, F.Cu at (170.8, 79.7)
- added REF**: MountingHole_3.2mm_M3, MountingHole:MountingHole_3.2mm_M3, F.Cu at (170.6, 116.6)
- added REF**: MountingHole_3.2mm_M3, MountingHole:MountingHole_3.2mm_M3, F.Cu at (114.3, 116.6)
