File: Inverter/Separator_filtr_skladowa_stala.kicad_pcb (KiCad board)
At the start: 2 copper layers, 70 x 40 mm, 40 parts, among them J1 Conn_Coaxial, J3 Conn_Coaxial, J5 Power, U1 ADA4622-2xCP, U2 ADA4622-2xCP

Commit message: pcb update
Parts:
- moved J3 30.3 mm to (154.4, 98.4), turned to 180 degrees
- moved H2 30.0 mm to (155.5, 83.5)
- moved H4 30.0 mm to (155.5, 113.5)
- moved U1 25.8 mm to (146.2, 98.2)
- moved C3 25.5 mm to (141.0, 98.5)
- moved C1 20.0 mm to (154.0, 104.5)
- moved R10 20.0 mm to (150.0, 104.5)
- moved R13 20.0 mm to (154.0, 108.0)
- moved R9 20.0 mm to (150.0, 108.0)
- moved C9 17.3 mm to (146.5, 89.4)
- moved C10 17.1 mm to (146.5, 87.0)
- moved C11 17.0 mm to (146.5, 84.5)
- moved C12 17.0 mm to (146.5, 82.0)
- moved RV1 16.0 mm to (142.0, 113.5)
- moved J5 15.5 mm to (142.5, 82.5)
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Routing:
- net +15V: track 46.1 -> 26.4 mm
- net -15V: track 37.3 -> 20.7 mm, vias 4 -> 0
- net Net-(R13-Pad1): track 36.9 -> 25.0 mm
- net Net-(U2A--): track 41.8 -> 30.0 mm
- net Net-(C4-Pad2): track 23.0 -> 15.5 mm, vias 0 -> 2
- net Net-(C1-Pad2): track 8.84 -> 12.4 mm
- net Net-(C2-Pad2): track 27.1 -> 23.7 mm
- net Net-(R5-Pad2): track 22.8 -> 25.5 mm
- net Net-(U1B--): track 13.0 -> 11.8 mm
- net Net-(J3-In): track 28.9 -> 27.9 mm
- net Net-(U2A-+): track 5.85 -> 5.00 mm
- net GND: track 0.89 -> 0.09 mm
- net Net-(R7-Pad2): track 2.50 -> 2.00 mm
- net Net-(U1A--): track 26.6 -> 27.0 mm, vias 0 -> 1
- net (no net): vias 0 -> 1
Other:
- board size 70 x 40 mm -> 40 x 40 mm

Commit message: Edit PCB
Connections:
- J1 pad 3: (no net) -> GND
- J1 pad 4: (no net) -> GND
- J1 pad 5: (no net) -> GND
- J3 pad 3: (no net) -> GND
- J3 pad 4: (no net) -> GND
- J3 pad 5: (no net) -> GND
Routing:
- net GND: track 0.09 -> 28.6 mm
- net Net-(U1A--): track 27.0 -> 24.7 mm, vias 1 -> 0
- net Net-(U1B--): track 11.8 -> 13.4 mm
- net Net-(U2A--): track 30.0 -> 30.3 mm, vias 2 -> 4
- net (no net): vias 1 -> 0

Commit message: pcb final version
Parts:
- added G***: LOGO, NaMi_logo:NaMi_logo, F.Cu at (151.0, 92.0)
- added R1: 100R, Resistor_SMD:R_0805_2012Metric_Pad1.20x1.40mm_HandSolder, F.Cu at (147.0, 116.5)
- added R18: 300R, Resistor_SMD:R_0805_2012Metric_Pad1.20x1.40mm_HandSolder, F.Cu at (159.0, 105.0)
- moved C4 10.5 mm to (146.5, 105.5), turned to 90 degrees
- moved R12 5.52 mm to (138.5, 105.5), turned to 90 degrees
- moved R16 4.03 mm to (143.5, 105.5), turned to 90 degrees
- moved R2 1.35 mm to (133.5, 93.0)
- moved U1 1.22 mm to (146.2, 99.4)
- moved R11 1.12 mm to (141.0, 105.5), turned to -90 degrees
- moved R15 1.12 mm to (144.5, 108.5)
- moved R17 1.00 mm to (126.0, 92.5)
- moved R5 1.00 mm to (131.5, 113.0)
- moved R6 1.00 mm to (131.5, 109.5)
Connections:
- C3 pad 2: Net-(J3-In) -> Net-(C3-Pad2)
- R15 pad 1: Net-(J3-In) -> Net-(C3-Pad2)
- RV1 pad 1: Net-(U2A--) -> Net-(R1-Pad1)
- U1 pad 7: Net-(J3-In) -> Net-(C3-Pad2)
Routing:
- net Net-(C3-Pad2): track 0.00 -> 32.4 mm, vias 0 -> 4
- net Net-(J3-In): track 28.3 -> 9.01 mm, vias 4 -> 2
- net Net-(U2A--): track 30.3 -> 38.8 mm, vias 4 -> 2
- net Net-(C4-Pad2): track 15.5 -> 8.07 mm, vias 2 -> 0
- net Net-(R1-Pad1): track 0.00 -> 6.43 mm
- net Net-(R13-Pad1): track 25.0 -> 29.0 mm, vias 0 -> 2
- net -15V: track 20.7 -> 23.6 mm, vias 0 -> 2
- net Net-(U1A--): track 24.7 -> 27.5 mm, vias 0 -> 2
- net Net-(U2A-+): track 5.00 -> 6.94 mm
- net Net-(R5-Pad2): track 25.5 -> 27.1 mm
- net +15V: track 26.1 -> 27.4 mm
- net Net-(J1-In): track 6.05 -> 7.05 mm
- net Net-(U1B--): track 13.4 -> 14.1 mm
- net Net-(C1-Pad2): track 12.4 -> 11.8 mm
- net Net-(C2-Pad2): track 23.7 -> 24.2 mm
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