File: Inverter/Separator_filtr_skladowa_stala.kicad_sch (KiCad schematic)
At the start: 40 parts, among them J1 Conn_Coaxial, J3 Conn_Coaxial, J5 Power, U1 ADA4622-2xCP, U2 ADA4622-2xCP

Commit message: pcb update
Other:
- note added: "Otwory mocujące"
- moved on the sheet: H1, H2, H3, H4
Changed lines of the file:
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@@
 	(generator_version "9.0")
 	(paper "A4")
+	(text "Otwory mocujące"
+		(exclude_from_sim no)
+		(at 29.21 162.814 0)
+		(effects
+			(font
+				(size 1.27 1.27)
+			)
+		)
+	)
 	(text "Blok zasilania"
 		(exclude_from_sim no)
@@
 	)
 	(junction
+		(at 29.21 184.15)
+		(diameter 0)
+		(color 0 0 0 0)
+	)
+	(junction
 		(at 227.33 31.75)
 		(diameter 0)
@@
 	)
 	(junction
-		(at 88.9 102.87)
+		(at 29.21 173.99)
 		(diameter 0)
 		(color 0 0 0 0)
 	)
 	(junction
-		(at 162.56 124.46)
+		(at 88.9 102.87)
 		(diameter 0)
 		(color 0 0 0 0)
 	)
 	(junction
-		(at 260.35 50.8)
+		(at 162.56 124.46)
 		(diameter 0)
 		(color 0 0 0 0)
 	)
 	(junction
-		(at 46.99 185.42)
+		(at 260.35 50.8)
 		(diameter 0)
 		(color 0 0 0 0)
@@
 	)
 	(junction
-		(at 46.99 175.26)
-		(diameter 0)
-		(color 0 0 0 0)
-	)
-	(junction
 		(at 222.25 31.75)
 		(diameter 0)
@@
 		)
 	)
+	(polyline
+		(pts
+			(xy 47.625 160.02) (xy 47.625 198.12)
+		)
+		(stroke
+			(width 0)
+			(type dash)
+			(color 255 0 0 1)
+		)
+	)
 	(wire
 		(pts
@@
 	(wire
 		(pts
+			(xy 29.21 184.15) (xy 34.29 184.15)
+		)
+		(stroke
+			(width 0)
+			(type default)
+		)
+	)
+	(wire
+		(pts
 			(xy 215.9 24.13) (xy 222.25 24.13)
 		)
@@
 	(wire
 		(pts
-			(xy 46.99 175.26) (xy 46.99 185.42)
+			(xy 29.21 173.99) (xy 29.21 184.15)
 		)
 		(stroke
@@
 	(wire
 		(pts
-			(xy 40.64 175.26) (xy 46.99 175.26)
+			(xy 24.13 173.99) (xy 29.21 173.99)
 		)
 		(stroke
@@
 	(wire
 		(pts
-			(xy 46.99 185.42) (xy 46.99 189.23)
+			(xy 29.21 184.15) (xy 29.21 187.96)
 		)
 		(stroke
@@
 		)
 	)
+	(polyline
+		(pts
+			(xy 12.065 160.02) (xy 47.625 160.02)
+		)
+		(stroke
+			(width 0)
+			(type dash)
+			(color 255 0 0 1)
+		)
+	)
 	(wire
 		(pts
@@
 	(wire
 		(pts
-			(xy 40.64 185.42) (xy 46.99 185.42)
+			(xy 24.13 184.15) (xy 29.21 184.15)
 		)
 		(stroke
@@
 		)
 	)
-	(wire
-		(pts
-			(xy 46.99 185.42) (xy 52.07 185.42)
-		)
-		(stroke
-			(width 0)
-			(type default)
-		)
-	)
 	(polyline
 		(pts
@@
 	(wire
 		(pts
-			(xy 109.22 121.92) (xy 111.76 121.92)
+			(xy 29.21 173.99) (xy 34.29 173.99)
 		)
 		(stroke
@@
 	(wire
 		(pts
-			(xy 260.35 50.8) (xy 271.78 50.8)
+			(xy 109.22 121.92) (xy 111.76 121.92)
 		)
 		(stroke
@@
 	(wire
 		(pts
-			(xy 147.32 137.16) (xy 147.32 127)
+			(xy 260.35 50.8) (xy 271.78 50.8)
 		)
 		(stroke
@@
 	(wire
 		(pts
-			(xy 29.21 36.83) (xy 31.75 36.83)
+			(xy 147.32 137.16) (xy 147.32 127)
 		)
 		(stroke
@@
 	(wire
 		(pts
-			(xy 162.56 124.46) (xy 167.64 124.46)
+			(xy 29.21 36.83) (xy 31.75 36.83)
 		)
 		(stroke
@@
 	(wire
 		(pts
-			(xy 189.23 104.14) (xy 210.82 104.14)
+			(xy 162.56 124.46) (xy 167.64 124.46)
 		)
 		(stroke
@@
 	(wire
 		(pts
-			(xy 76.2 119.38) (xy 81.28 119.38)
+			(xy 189.23 104.14) (xy 210.82 104.14)
 		)
 		(stroke
@@
 	(wire
 		(pts
-			(xy 76.2 106.68) (xy 76.2 119.38)
+			(xy 76.2 119.38) (xy 81.28 119.38)
 		)
 		(stroke
@@
 	(wire
 		(pts
-			(xy 46.99 175.26) (xy 52.07 175.26)
+			(xy 76.2 106.68) (xy 76.2 119.38)
 		)
 		(stroke
@@
 	(symbol
 		(lib_id "power:GND")
-		(at 46.99 189.23 0)
+		(at 29.21 187.96 0)
 		(unit 1)
 		(exclude_from_sim no)
@@
 		(fields_autoplaced yes)
 		(property "Reference" "#PWR027"
-			(at 46.99 195.58 0)
+			(at 29.21 194.31 0)
 			(effects
 				(font
@@
 		)
 		(property "Value" "GND"
-			(at 46.99 194.31 0)
+			(at 29.21 193.04 0)
 			(effects
 				(font
@@
 		)
 		(property "Footprint" ""
-			(at 46.99 189.23 0)
+			(at 29.21 187.96 0)
 			(effects
 				(font
@@
 		)
 		(property "Datasheet" ""
-			(at 46.99 189.23 0)
+			(at 29.21 187.96 0)
 			(effects
 				(font
@@
 		)
 		(property "Description" "Power symbol creates a global label with name \"GND\" , ground"
-			(at 46.99 189.23 0)
+			(at 29.21 187.96 0)
 			(effects
 				(font
@@
 	(symbol
 		(lib_id "Mechanical:MountingHole_Pad")
-		(at 40.64 182.88 0)
+		(at 24.13 181.61 0)
 		(unit 1)
 		(exclude_from_sim no)
@@
 		(fields_autoplaced yes)
 		(property "Reference" "H3"
-			(at 43.18 180.3399 0)
+			(at 26.67 179.0699 0)
 			(effects
 				(font
@@
 		)
 		(property "Value" "MountingHole_Pad"
-			(at 43.18 182.8799 0)
+			(at 26.67 181.6099 0)
 			(effects
 				(font
@@
 		)
 		(property "Footprint" "MountingHole:MountingHole_3.2mm_M3_DIN965_Pad"
-			(at 40.64 182.88 0)
+			(at 24.13 181.61 0)
 			(effects
 				(font
@@
 		)
 		(property "Datasheet" "~"
-			(at 40.64 182.88 0)
+			(at 24.13 181.61 0)
 			(effects
 				(font
@@
 		)
 		(property "Description" "Mounting Hole with connection"
-			(at 40.64 182.88 0)
+			(at 24.13 181.61 0)
 			(effects
 				(font
@@
 	(symbol
 		(lib_id "Mechanical:MountingHole_Pad")
-		(at 52.07 182.88 0)
+		(at 34.29 181.61 0)
 		(unit 1)
 		(exclude_from_sim no)
@@
 		(fields_autoplaced yes)
 		(property "Reference" "H4"
-			(at 54.61 180.3399 0)
+			(at 36.83 179.0699 0)
 			(effects
 				(font
@@
 		)
 		(property "Value" "MountingHole_Pad"
-			(at 54.61 182.8799 0)
+			(at 36.83 181.6099 0)
 			(effects
 				(font
@@
 		)
 		(property "Footprint" "MountingHole:MountingHole_3.2mm_M3_DIN965_Pad"
-			(at 52.07 182.88 0)
+			(at 34.29 181.61 0)
 			(effects
 				(font
@@
 		)
 		(property "Datasheet" "~"
-			(at 52.07 182.88 0)
+			(at 34.29 181.61 0)
 			(effects
 				(font
@@
 		)
 		(property "Description" "Mounting Hole with connection"
-			(at 52.07 182.88 0)
+			(at 34.29 181.61 0)
 			(effects
 				(font
@@
 	(symbol
 		(lib_id "Mechanical:MountingHole_Pad")
-		(at 40.64 172.72 0)
+		(at 24.13 171.45 0)
 		(unit 1)
 		(exclude_from_sim no)
@@
 		(fields_autoplaced yes)
 		(property "Reference" "H1"
-			(at 43.18 170.1799 0)
+			(at 26.67 168.9099 0)
 			(effects
 				(font
@@
 		)
 		(property "Value" "MountingHole_Pad"
-			(at 43.18 172.7199 0)
+			(at 26.67 171.4499 0)
 			(effects
 				(font
@@
 		)
 		(property "Footprint" "MountingHole:MountingHole_3.2mm_M3_DIN965_Pad"
-			(at 40.64 172.72 0)
+			(at 24.13 171.45 0)
 			(effects
 				(font
@@
 		)
 		(property "Datasheet" "~"
-			(at 40.64 172.72 0)
+			(at 24.13 171.45 0)
 			(effects
 				(font
@@
 		)
 		(property "Description" "Mounting Hole with connection"
-			(at 40.64 172.72 0)
+			(at 24.13 171.45 0)
 			(effects
 				(font
@@
 	(symbol
 		(lib_id "Mechanical:MountingHole_Pad")
-		(at 52.07 172.72 0)
+		(at 34.29 171.45 0)
 		(unit 1)
 		(exclude_from_sim no)
@@
 		(fields_autoplaced yes)
 		(property "Reference" "H2"
-			(at 54.61 170.1799 0)
+			(at 36.83 168.9099 0)
 			(effects
 				(font
@@
 		)
 		(property "Value" "MountingHole_Pad"
-			(at 54.61 172.7199 0)
+			(at 36.83 171.4499 0)
 			(effects
 				(font
@@
 		)
 		(property "Footprint" "MountingHole:MountingHole_3.2mm_M3_DIN965_Pad"
-			(at 52.07 172.72 0)
+			(at 34.29 171.45 0)
 			(effects
 				(font
@@
 		)
 		(property "Datasheet" "~"
-			(at 52.07 172.72 0)
+			(at 34.29 171.45 0)
 			(effects
 				(font
@@
 		)
 		(property "Description" "Mounting Hole with connection"
-			(at 52.07 172.72 0)
+			(at 34.29 171.45 0)
 			(effects
 				(font

Commit message: pcb final version
Parts:
- added R1: 100R, Resistor_SMD:R_0805_2012Metric_Pad1.20x1.40mm_HandSolder, symbol Device:R
- added R18: 300R, Resistor_SMD:R_0805_2012Metric_Pad1.20x1.40mm_HandSolder, symbol Device:R
Connections:
- net at C3.2, R15.1, U1.7: now also R18.1; no longer J3.1 (In)
- net at R17.2, U2.2 (-): now also R1.2; no longer RV1.1
- new net: J3.1 (In), R18.2
- new net: R1.1, RV1.1
Other:
- moved on the sheet: J3
Changed lines of the file:
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@@
 	)
 	(junction
-		(at 146.05 102.87)
+		(at 228.6 127)
 		(diameter 0)
 		(color 0 0 0 0)
 	)
 	(junction
-		(at 76.2 119.38)
+		(at 146.05 102.87)
 		(diameter 0)
 		(color 0 0 0 0)
 	)
 	(junction
-		(at 228.6 127)
+		(at 260.35 58.42)
 		(diameter 0)
 		(color 0 0 0 0)
 	)
 	(junction
-		(at 260.35 58.42)
+		(at 76.2 119.38)
 		(diameter 0)
 		(color 0 0 0 0)
@@
 	(wire
 		(pts
-			(xy 81.28 106.68) (xy 76.2 106.68)
-		)
-		(stroke
-			(width 0)
-			(type default)
-		)
-	)
-	(wire
-		(pts
 			(xy 222.25 31.75) (xy 227.33 31.75)
 		)
@@
 	(wire
 		(pts
+			(xy 76.2 115.57) (xy 76.2 119.38)
+		)
+		(stroke
+			(width 0)
+			(type default)
+		)
+	)
+	(wire
+		(pts
 			(xy 123.19 121.92) (xy 123.19 120.65)
 		)
@@
 	(wire
 		(pts
+			(xy 76.2 119.38) (xy 81.28 119.38)
+		)
+		(stroke
+			(width 0)
+			(type default)
+		)
+	)
+	(wire
+		(pts
 			(xy 123.19 137.16) (xy 123.19 135.89)
 		)
@@
 	(wire
 		(pts
+			(xy 241.3 132.08) (xy 241.3 134.62)
+		)
+		(stroke
+			(width 0)
+			(type default)
+		)
+	)
+	(wire
+		(pts
 			(xy 255.27 50.8) (xy 260.35 50.8)
 		)
@@
 	(wire
 		(pts
+			(xy 76.2 107.95) (xy 76.2 106.68)
+		)
+		(stroke
+			(width 0)
+			(type default)
+		)
+	)
+	(wire
+		(pts
 			(xy 82.55 48.26) (xy 82.55 52.07)
 		)
@@
 	(wire
 		(pts
-			(xy 59.69 119.38) (xy 63.5 119.38)
+			(xy 76.2 106.68) (xy 81.28 106.68)
 		)
 		(stroke
@@
 	(wire
 		(pts
-			(xy 16.51 34.29) (xy 31.75 34.29)
+			(xy 59.69 119.38) (xy 63.5 119.38)
 		)
 		(stroke
@@
 	(wire
 		(pts
-			(xy 233.68 132.08) (xy 233.68 133.985)
+			(xy 16.51 34.29) (xy 31.75 34.29)
 		)
 		(stroke
@@
 	(wire
 		(pts
-			(xy 76.2 119.38) (xy 81.28 119.38)
-		)
-		(stroke
-			(width 0)
-			(type default)
-		)
-	)
-	(wire
-		(pts
-			(xy 76.2 106.68) (xy 76.2 119.38)
-		)
-		(stroke
-			(width 0)
-			(type default)
-		)
-	)
-	(wire
-		(pts
 			(xy 165.1 40.64) (xy 186.69 40.64)
 		)
@@
 	(symbol
 		(lib_id "power:GND")
-		(at 233.68 133.985 0)
+		(at 241.3 134.62 0)
 		(unit 1)
 		(exclude_from_sim no)
@@
 		(fields_autoplaced yes)
 		(property "Reference" "#PWR014"
-			(at 233.68 140.335 0)
+			(at 241.3 140.97 0)
 			(effects
 				(font
@@
 		)
 		(property "Value" "GND"
-			(at 233.68 139.065 0)
+			(at 241.3 139.7 0)
 			(effects
 				(font
@@
 		)
 		(property "Footprint" ""
-			(at 233.68 133.985 0)
+			(at 241.3 134.62 0)
 			(effects
 				(font
@@
 		)
 		(property "Datasheet" ""
-			(at 233.68 133.985 0)
+			(at 241.3 134.62 0)
 			(effects
 				(font
@@
 		)
 		(property "Description" "Power symbol creates a global label with name \"GND\" , ground"
-			(at 233.68 133.985 0)
+			(at 241.3 134.62 0)
 			(effects
 				(font
@@
 	)
 	(symbol
+		(lib_id "Device:R")
+		(at 232.41 127 90)
+		(unit 1)
+		(exclude_from_sim no)
+		(in_bom yes)
+		(on_board yes)
+		(dnp no)
+		(fields_autoplaced yes)
+		(property "Reference" "R18"
+			(at 232.41 120.65 90)
+			(effects
+				(font
+					(size 1.27 1.27)
+				)
+			)
+		)
+		(property "Value" "300R"
+			(at 232.41 123.19 90)
+			(effects
+				(font
+					(size 1.27 1.27)
+				)
+			)
+		)
+		(property "Footprint" "Resistor_SMD:R_0805_2012Metric_Pad1.20x1.40mm_HandSolder"
+			(at 232.41 128.778 90)
+			(effects
+				(font
+					(size 1.27 1.27)
+				)
+				(hide yes)
+			)
+		)
+		(property "Datasheet" "~"
+			(at 232.41 127 0)
+			(effects
+				(font
+					(size 1.27 1.27)
+				)
+				(hide yes)
+			)
+		)
+		(property "Description" "Resistor"
+			(at 232.41 127 0)
+			(effects
+				(font
+					(size 1.27 1.27)
+				)
+				(hide yes)
+			)
+		)
+		(pin "1"
+		)
+		(pin "2"
+		)
+		(instances
+			(project ""
+				(path "/483bf3cf-81ef-401a-a7d9-4215728deaac"
+					(reference "R18")
+					(unit 1)
+				)
+			)
+		)
+	)
+	(symbol
 		(lib_id "Connector:Conn_Coaxial")
-		(at 233.68 127 0)
+		(at 241.3 127 0)
 		(unit 1)
 		(exclude_from_sim no)
@@
 		(dnp no)
 		(property "Reference" "J3"
-			(at 237.49 126.0231 0)
+			(at 245.11 126.0231 0)
 			(effects
 				(font
@@
 		)
 		(property "Value" "Conn_Coaxial"
-			(at 237.49 128.5631 0)
+			(at 245.11 128.5631 0)
 			(effects
 				(font
@@
 		)
 		(property "Footprint" "CONN SMA JACK STR 50 OHM SMD:CONN_732511350_MOL"
-			(at 233.68 127 0)
+			(at 241.3 127 0)
 			(effects
 				(font
@@
 		)
 		(property "Datasheet" "~"
-			(at 233.68 127 0)
+			(at 241.3 127 0)
 			(effects
 				(font
@@
 		)
 		(property "Description" "coaxial connector (BNC, SMA, SMB, SMC, Cinch/RCA, LEMO, ...)"
-			(at 233.68 127 0)
+			(at 241.3 127 0)
 			(effects
 				(font
@@
 					(unit 1)
 				)
+			)
+		)
+	)
+	(symbol
+		(lib_id "Device:R")
+		(at 76.2 111.76 0)
+		(unit 1)
+		(exclude_from_sim no)
+		(in_bom yes)
+		(on_board yes)
+		(dnp no)
+		(property "Reference" "R1"
+			(at 77.724 110.49 0)
+			(effects
+				(font
+					(size 1.27 1.27)
+				)
+				(justify left)
+			)
+		)
+		(property "Value" "100R"
+			(at 77.47 113.03 0)
+			(effects
+				(font
+					(size 1.27 1.27)
+				)
+				(justify left)
+			)
+		)
+		(property "Footprint" "Resistor_SMD:R_0805_2012Metric_Pad1.20x1.40mm_HandSolder"
+			(at 74.422 111.76 90)
+			(effects
+				(font
+					(size 1.27 1.27)
+				)
+				(hide yes)
+			)
+		)
+		(property "Datasheet" "~"
+			(at 76.2 111.76 0)
+			(effects
+				(font
+					(size 1.27 1.27)
+				)
+				(hide yes)
+			)
+		)
+		(property "Description" "Resistor"
+			(at 76.2 111.76 0)
+			(effects
+				(font
+					(size 1.27 1.27)
+				)
+				(hide yes)
+			)
+		)
+		(pin "2"
+		)
+		(pin "1"
+		)
+		(instances
+			(project ""
+				(path "/483bf3cf-81ef-401a-a7d9-4215728deaac"
+					(reference "R1")
+					(unit 1)
+				)
